Commit message: updated with gazebo startup errors and warnings reduced in size

File: igvc_description/models/robots/iggy_base.urdf.xacro (robot description, xacro)
@@ -20,11 +20,11 @@
     <property name="wheel_offset_z_from_base_link" value="-${wheel_radius_big}" />
     <macro name="iggy_base_macro">
-        <!-- Links and Joints (i.e., the robot) -->
-        <link name="base_footprint"/>
+        <!-- Links and Joints (i.e., the robot)
+        <link name="base_link"/>
         <joint name="bf_to_bl" type="fixed">
           <origin xyz="0.0 0.0 -${base_size_z * 2}" rpy="0.0 0.0 0.0" />
           <parent link="base_link"/>
           <child link="base_footprint"/>
-        </joint>
+        </joint> -->
         <link name="base_link">
             <inertial>
@@ -71,4 +71,5 @@
         <plugin name="diffdrive_plugin_multiwheel" filename="libdiffdrive_plugin_multi_wheel.so">
                 <alwaysOn>true</alwaysOn>
+            <robotNamespace>roboteq_driver</robotNamespace>
                 <updateRate>50.0</updateRate>
                 <leftJoints>left_0_wheel_joint left_1_wheel_joint left_2_wheel_joint left_3_wheel_joint left_4_wheel_joint left_5_wheel_joint</leftJoints>
@@ -80,5 +81,6 @@
                 <robotNamespace>/</robotNamespace>
                 <robotBaseFrame>base_link</robotBaseFrame>
-                <commandTopic>/iggy/cmd_vel</commandTopic>
+                <odometryFrame>odom</odometryFrame>
+                <commandTopic>/roboteq_driver/cmd_vel</commandTopic>
                 <publishOdometryTf>1</publishOdometryTf>
                 <publishOdometryMsg>1</publishOdometryMsg>
@@ -99,5 +101,5 @@
           <updateRate>50.0</updateRate>
           <bodyName>base_link</bodyName>
-          <topicName>/iggy/imu_quat</topicName>
+          <topicName>/imu/data</topicName>
           <accelDrift>0.0 0.0 0.0</accelDrift>
           <accelGaussianNoise>0.1 0.1 0.1</accelGaussianNoise>
@@ -109,4 +111,5 @@
         <plugin name="gps_controller" filename="libhector_gazebo_ros_gps.so">
             <alwayson>1</alwayson>
+            <robotNamespace>gps</robotNamespace>
             <updaterate>10.0</updaterate>
             <bodyname>base_link</bodyname>

File: igvc_description/urdf/igvc.urdf.xacro (robot description, xacro)
@@ -3,9 +3,10 @@
     xmlns:sensor="http://playerstage.sourceforge.net/gazebo/xmlschema/#sensor"
     xmlns:controller="http://playerstage.sourceforge.net/gazebo/xmlschema/#controller"
-    xmlns:interface="http://playerstage.sourceforge.net/gazebo/xmlschema/#interface">
+    xmlns:interface="http://playerstage.sourceforge.net/gazebo/xmlschema/#interface"
+    xmlns:xacro="http://playerstage.sourceforge.net/gazebo/xmlschema/#interface">
     <!-- Included URDF Files -->
-    <include filename="$(find igvc_description)/models/robots/iggy_base.urdf.xacro" />
-    <include filename="$(find usma_velodyne)/urdf/velodyne.urdf.xacro" />
-    <include filename="$(find pointgrey_camera_description)/urdf/pointgrey_bumblebee2.urdf.xacro" />
+    <xacro:include filename="$(find igvc_description)/models/robots/iggy_base.urdf.xacro" />
+    <xacro:include filename="$(find usma_velodyne)/urdf/velodyne.urdf.xacro" />
+<!--    <xacro:include filename="$(find pointgrey_camera_description)/urdf/pointgrey_bumblebee2.urdf.xacro" />-->
     <iggy_base_macro />
     <plexiglass_mount_macro />
@@ -16,4 +17,5 @@
     <!--velodyne_32 parent="base_link" prefix="v32"  vb_x="0.0" vb_y="0.0" vb_z="0.5" vb_r="0.0" vb_p="0.0" vb_yaw="0.0" /-->
     <velodyne_32_w_mast parent_frame="base_link" parent_link="velodyne_mount" prefix="v32" />
+<!--
     <joint name="bumblebee2_camera_joint" type="fixed">
       <origin xyz="0.25 0 0"
@@ -22,4 +24,5 @@
       <child link="bumblebee2" />
     </joint>
+-->
     <link name="imu" />
     <joint name="imu_joint" type="fixed">
